Commit message: Added urdf files

File: atlas_description/urdf/chassis.urdf.xacro (robot description, xacro)
@@ -1,7 +1,7 @@
 <?xml version="1.0"?>
-<robot name="right_track" xmlns:xacro="http://ros.org/wiki/xacro">
-  <xacro:property name="right_track_mesh" value="package://atlas_description/meshes/visual_model/right_track.dae"/>
-  <xacro:property name="right_track_collision_mesh" value="package://atlas_description/meshes/collision_model/right_track_collision.dae"/>
-  <xacro:macro name="right_track_inertial" params="mass">
+<robot name="chassis" xmlns:xacro="http://ros.org/wiki/xacro">
+  <xacro:property name="atlas_chassis_mesh" value="package://atlas_description/meshes/visual_model/chassis.dae"/>
+  <xacro:property name="atlas_chassis_collision_mesh" value="package://atlas_description/meshes/collision_model/chassis.dae"/>
+  <xacro:macro name="atlas_chassis_inertial" params="mass">
     <inertial>
       <mass value="${mass}" />
@@ -9,9 +9,9 @@
     </inertial>
   </xacro:macro>
-  <xacro:macro name="atlas_right_track" params="prefix parent mass link_xyz link_rpy joint_xyz joint_rpy">
+  <xacro:macro name="atlas_chassis" params="prefix parent mass link_xyz link_rpy joint_xyz joint_rpy">
     <link name="${prefix}_link">
       <visual>
         <geometry>
-          <mesh filename="${right_track_mesh}"/>
+          <mesh filename="${atlas_chassis_mesh}"/>
         </geometry>
         <origin xyz="${link_xyz}" rpy="${link_rpy}"/>
@@ -19,9 +19,9 @@
       <collision>
         <geometry>
-          <mesh filename="${right_track_collision_mesh}"/>
+          <mesh filename="${atlas_chassis_collision_mesh}"/>
         </geometry>
         <origin xyz="${link_xyz}" rpy="${link_rpy}"/>
       </collision>
-      <xacro:right_track_inertial mass="${mass}"/>
+      <xacro:atlas_chassis_inertial mass="${mass}"/>
     </link>
     <joint name="${prefix}_joint" type="fixed">
